File: conn_and_power.kicad_sch (KiCad schematic)
At the start: 5 parts, among them J4 Interconnect, U3 LP5907MFX-3.3

Commit message: update component assignments
Parts:
- C25, C26: footprint Capacitor_SMD:C_0603_1608Metric -> Capacitor_SMD:C_0805_2012Metric
Changed lines of the file:
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@@
 			)
 		)
-		(property "Footprint" "Capacitor_SMD:C_0603_1608Metric"
+		(property "Footprint" "Capacitor_SMD:C_0805_2012Metric"
 			(at 121.92 82.55 0)
 			(effects
@@
 			)
 		)
-		(property "Footprint" "Capacitor_SMD:C_0603_1608Metric"
+		(property "Footprint" "Capacitor_SMD:C_0805_2012Metric"
 			(at 156.21 82.55 0)
 			(effects

Commit message: sync pcb
Parts:
- C29: renamed from C25; value 1uF -> 1μF
- C30: renamed from C26; value 1uF -> 1μF
Changed lines of the file:
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@@
 		(dnp no)
 		(fields_autoplaced yes)
-		(property "Reference" "#FLG02"
+		(property "Reference" "#FLG03"
 			(at 77.47 66.675 0)
 			(effects
@@
 			(project "mv2_taa3040"
 				(path "/41a55a1d-5108-482f-b313-9eaa5d011dff/cad1070f-df9f-433f-9c9e-3f26e05af870"
-					(reference "#FLG02")
+					(reference "#FLG03")
 					(unit 1)
 				)
@@
 		(on_board yes)
 		(dnp no)
-		(property "Reference" "#PWR056"
+		(property "Reference" "#PWR059"
 			(at 87.63 104.14 0)
 			(effects
@@
 			(project "mv2_taa3040"
 				(path "/41a55a1d-5108-482f-b313-9eaa5d011dff/cad1070f-df9f-433f-9c9e-3f26e05af870"
-					(reference "#PWR056")
+					(reference "#PWR059")
 					(unit 1)
 				)
@@
 		(dnp no)
 		(fields_autoplaced yes)
-		(property "Reference" "#FLG03"
+		(property "Reference" "#FLG04"
 			(at 80.01 66.675 0)
 			(effects
@@
 			(project "mv2_taa3040"
 				(path "/41a55a1d-5108-482f-b313-9eaa5d011dff/cad1070f-df9f-433f-9c9e-3f26e05af870"
-					(reference "#FLG03")
+					(reference "#FLG04")
 					(unit 1)
 				)
@@
 		(dnp no)
 		(fields_autoplaced yes)
-		(property "Reference" "#FLG04"
+		(property "Reference" "#FLG02"
 			(at 74.93 127.635 0)
 			(effects
@@
 			(project "mv2_taa3040"
 				(path "/41a55a1d-5108-482f-b313-9eaa5d011dff/cad1070f-df9f-433f-9c9e-3f26e05af870"
-					(reference "#FLG04")
+					(reference "#FLG02")
 					(unit 1)
 				)
@@
 		(dnp no)
 		(fields_autoplaced yes)
-		(property "Reference" "#PWR060"
+		(property "Reference" "#PWR057"
 			(at 77.47 86.36 0)
 			(effects
@@
 			(project "mv2_taa3040"
 				(path "/41a55a1d-5108-482f-b313-9eaa5d011dff/cad1070f-df9f-433f-9c9e-3f26e05af870"
-					(reference "#PWR060")
+					(reference "#PWR057")
 					(unit 1)
 				)
@@
 		(dnp no)
 		(fields_autoplaced yes)
-		(property "Reference" "#PWR057"
+		(property "Reference" "#PWR060"
 			(at 87.63 121.92 0)
 			(effects
@@
 			(project "mv2_taa3040"
 				(path "/41a55a1d-5108-482f-b313-9eaa5d011dff/cad1070f-df9f-433f-9c9e-3f26e05af870"
-					(reference "#PWR057")
+					(reference "#PWR060")
 					(unit 1)
 				)
@@
 		(dnp no)
 		(fields_autoplaced yes)
-		(property "Reference" "#PWR059"
+		(property "Reference" "#PWR056"
 			(at 77.47 76.2 0)
 			(effects
@@
 			(project ""
 				(path "/41a55a1d-5108-482f-b313-9eaa5d011dff/cad1070f-df9f-433f-9c9e-3f26e05af870"
-					(reference "#PWR059")
+					(reference "#PWR056")
 					(unit 1)
 				)
@@
 		(on_board yes)
 		(dnp no)
-		(property "Reference" "C25"
+		(property "Reference" "C29"
 			(at 121.92 80.01 0)
 			(effects
@@
 			)
 		)
-		(property "Value" "1uF"
+		(property "Value" "1μF"
 			(at 121.92 85.09 0)
 			(effects
@@
 			(project "mv2_taa3040"
 				(path "/41a55a1d-5108-482f-b313-9eaa5d011dff/cad1070f-df9f-433f-9c9e-3f26e05af870"
-					(reference "C25")
+					(reference "C29")
 					(unit 1)
 				)
@@
 		(on_board yes)
 		(dnp no)
-		(property "Reference" "C26"
+		(property "Reference" "C30"
 			(at 156.21 80.01 0)
 			(effects
@@
 			)
 		)
-		(property "Value" "1uF"
+		(property "Value" "1μF"
 			(at 156.21 85.09 0)
 			(effects
@@
 			(project "mv2_taa3040"
 				(path "/41a55a1d-5108-482f-b313-9eaa5d011dff/cad1070f-df9f-433f-9c9e-3f26e05af870"
-					(reference "C26")
+					(reference "C30")
 					(unit 1)
 				)
@@
 		(dnp no)
 		(fields_autoplaced yes)
-		(property "Reference" "#PWR055"
+		(property "Reference" "#PWR058"
 			(at 87.63 88.9 0)
 			(effects
@@
 			(project "mv2_taa3040"
 				(path "/41a55a1d-5108-482f-b313-9eaa5d011dff/cad1070f-df9f-433f-9c9e-3f26e05af870"
-					(reference "#PWR055")
+					(reference "#PWR058")
 					(unit 1)
 				)
@@
 		(dnp no)
 		(fields_autoplaced yes)
-		(property "Reference" "#PWR058"
+		(property "Reference" "#PWR055"
 			(at 77.47 73.66 0)
 			(effects
@@
 			(project "mv2_taa3040"
 				(path "/41a55a1d-5108-482f-b313-9eaa5d011dff/cad1070f-df9f-433f-9c9e-3f26e05af870"
-					(reference "#PWR058")
-					(unit 1)
-				)
+					(reference "#PWR055")
+					(unit 1)
+				)
